File: boards/nf_ecp5_45/pcie.kicad_sch (KiCad schematic)
At the start: 17 parts, among them J2 Bus_PCI_Express_x4, U1 ECP5U_25_CABGA256, X1 SG-8002LB

Commit message: board
Connections:
- net USR_LED0: now reaches U1.P12 (PR47D/-/LRC_GPLL0C_IN/RDQ44)
- net USR_LED1: now reaches U1.P13 (PR41A/+/HS/RDQ44)
- net USR_LED2: now reaches U1.P14 (PR38B/-/HS/RDQ44)
Changed lines of the file:
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@@
+    )
+  )
+  (global_label "USR_LED1" (shape input) (at 183.769 104.648 180) (fields_autoplaced)
+    (effects (font (size 1.27 1.27)) (justify right))
+    (property "Intersheetrefs" "${INTERSHEET_REFS}" (at 171.3496 104.648 0)
+      (effects (font (size 1.27 1.27)) (justify right) hide)
     )
   )
@@
     )
   )
+  (global_label "USR_LED0" (shape input) (at 183.769 132.588 180) (fields_autoplaced)
+    (effects (font (size 1.27 1.27)) (justify right))
+    (property "Intersheetrefs" "${INTERSHEET_REFS}" (at 171.3496 132.588 0)
+      (effects (font (size 1.27 1.27)) (justify right) hide)
+    )
+  )
   (global_label "pcie_3v3_aux" (shape input) (at 105.41 62.611 90) (fields_autoplaced)
     (effects (font (size 1.27 1.27)) (justify left))
@@
     )
   )
+  (global_label "USR_LED2" (shape input) (at 183.769 97.028 180) (fields_autoplaced)
+    (effects (font (size 1.27 1.27)) (justify right))
+    (property "Intersheetrefs" "${INTERSHEET_REFS}" (at 171.3496 97.028 0)
+      (effects (font (size 1.27 1.27)) (justify right) hide)
+    )
+  )
