File: boards/nf_ecp5_45/led.kicad_sch (KiCad schematic)
At the start: 10 parts, among them Q1 2N7002_SOT-23-3, Q2 2N7002_SOT-23-3, Q3 2N7002_SOT-23-3

Commit message: test
Other:
- note added: "TODO: change colors, replace fpga_done"
- note added: "TODO: use 1k resistors"
Changed lines of the file:
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@@
+    (effects (font (size 1.27 1.27)) (justify left bottom))
+  )
+  (text "TODO: use 1k resistors" (at 47.371 71.501 0)
+    (effects (font (size 1.27 1.27)) (justify left bottom))
+  )
+  (text "TODO: change colors, replace fpga_done" (at 122.428 49.403 0)
     (effects (font (size 1.27 1.27)) (justify left bottom))
   )

Commit message: board
Parts:
- removed TP9: TestPoint, TestPoint:TestPoint_Pad_D1.0mm, symbol Connector:TestPoint
- D1: footprint LED_SMD:LED_0805_2012Metric -> LED_SMD:LED_0603_1608Metric; LCSC C34499 -> C5355421
- D2: footprint LED_SMD:LED_0805_2012Metric -> LED_SMD:LED_0603_1608Metric; LCSC C2297 -> C5179624
- D3: footprint LED_SMD:LED_0805_2012Metric -> LED_SMD:LED_0603_1608Metric; LCSC C2296 -> C22371297
- R33, R34, R5: value 200R -> 1k; LCSC C25087 -> C11702; Val 200R -> 1k
Connections:
- net FPGA_DONE renamed USR_LED2
Other:
- note added: "led parts 0603 (2024-09-04): red: C5179624 green: C22371297 blue: C5355421"
- note removed: "TODO: change colors, replace fpga_done"
- note removed: "TODO: change to basic parts: C84256, C2297, C2296"
- note removed: "TODO: check if 0 or 1"
- note removed: "TODO: use 1k resistors"
Changed lines of the file:
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@@
 (kicad_sch (version 20230121) (generator eeschema)
   (paper "A4")
-  (junction (at 156.21 121.285) (diameter 0) (color 0 0 0 0)
-  )
   (wire (pts (xy 163.195 50.8) (xy 172.085 50.8))
     (stroke (width 0) (type default))
@@
     (stroke (width 0) (type default))
   )
-  (wire (pts (xy 153.67 121.285) (xy 156.21 121.285))
-    (stroke (width 0) (type default))
-  )
-  (wire (pts (xy 156.21 116.078) (xy 156.21 121.285))
-    (stroke (width 0) (type default))
-  )
   (wire (pts (xy 163.195 50.8) (xy 163.195 52.07))
     (stroke (width 0) (type default))
@@
     (stroke (width 0) (type default))
   )
-  (wire (pts (xy 156.21 121.285) (xy 158.75 121.285))
+  (wire (pts (xy 153.67 121.285) (xy 158.75 121.285))
     (stroke (width 0) (type default))
   )
@@
     (stroke (width 0) (type default))
   )
-  (text "TODO: change to basic parts:\nC84256, C2297, C2296	\n"
-    (at 99.06 67.31 0)
+  (text "led parts 0603 (2024-09-04):\nred: C5179624\ngreen: C22371297\nblue: C5355421"
+    (at 71.501 62.103 0)
     (effects (font (size 1.27 1.27)) (justify left bottom))
-  )
-  (text "TODO: check if 0 or 1" (at 144.78 127.635 0)
-    (effects (font (size 1.27 1.27)) (justify left bottom))
-  )
-  (text "TODO: use 1k resistors" (at 47.371 71.501 0)
-    (effects (font (size 1.27 1.27)) (justify left bottom))
-  )
-  (text "TODO: change colors, replace fpga_done" (at 122.428 49.403 0)
-    (effects (font (size 1.27 1.27)) (justify left bottom))
-  )
-  (global_label "FPGA_DONE" (shape input) (at 153.67 121.285 180) (fields_autoplaced)
-    (effects (font (size 1.27 1.27)) (justify right))
-    (property "Intersheetrefs" "${INTERSHEET_REFS}" (at 139.92 121.285 0)
-      (effects (font (size 1.27 1.27)) (justify right) hide)
-    )
   )
   (global_label "VCC3V3" (shape input) (at 196.85 111.125 0) (fields_autoplaced)
@@
     )
   )
+  (global_label "USR_LED2" (shape input) (at 153.67 121.285 180) (fields_autoplaced)
+    (effects (font (size 1.27 1.27)) (justify right))
+    (property "Intersheetrefs" "${INTERSHEET_REFS}" (at 141.2506 121.285 0)
+      (effects (font (size 1.27 1.27)) (justify right) hide)
+    )
+  )
   (global_label "USR_LED0" (shape input) (at 55.245 92.71 180) (fields_autoplaced)
     (effects (font (size 1.27 1.27)) (justify right))
@@
         (path "/9bed7131-c603-46c6-ae3c-0e9faa418ea0/5d8c101e-63d8-417a-b55c-72ab74e8719b"
           (reference "#PWR048") (unit 1)
-        )
-      )
-    )
-  )
-  (symbol (lib_id "Connector:TestPoint") (at 156.21 116.078 0) (unit 1)
-    (in_bom yes) (on_board yes) (dnp no) (fields_autoplaced)
-    (property "Reference" "TP9" (at 158.75 111.506 0)
-      (effects (font (size 1.27 1.27)) (justify left))
-    )
-    (property "Value" "TestPoint" (at 158.75 114.046 0)
-      (effects (font (size 1.27 1.27)) (justify left))
-    )
-    (property "Footprint" "TestPoint:TestPoint_Pad_D1.0mm" (at 161.29 116.078 0)
-      (effects (font (size 1.27 1.27)) hide)
-    )
-    (property "Datasheet" "~" (at 161.29 116.078 0)
-      (effects (font (size 1.27 1.27)) hide)
-    )
-    (pin "1")
-    (instances
-      (project "nf_tpu"
-        (path "/9bed7131-c603-46c6-ae3c-0e9faa418ea0/5d8c101e-63d8-417a-b55c-72ab74e8719b"
-          (reference "TP9") (unit 1)
         )
       )
@@
       (effects (font (size 1.27 1.27) (thickness 0.15)) (justify left bottom) hide)
     )
-    (property "Footprint" "LED_SMD:LED_0805_2012Metric" (at 61.595 92.71 0)
+    (property "Footprint" "LED_SMD:LED_0603_1608Metric" (at 61.595 92.71 0)
       (effects (font (size 1.27 1.27) (thickness 0.15)) (justify left bottom) hide)
     )
@@
       (effects (font (size 1.27 1.27) (thickness 0.15)) (justify left bottom) hide)
     )
-    (property "LCSC" "C2297" (at 84.455 82.55 0)
+    (property "LCSC" "C5179624" (at 84.455 82.55 0)
       (effects (font (size 1.27 1.27)) hide)
     )
@@
       (effects (font (size 1.27 1.27)))
     )
-    (property "Value" "200R" (at 206.375 63.5 0)
+    (property "Value" "1k" (at 206.375 63.5 0)
       (effects (font (size 1.27 1.27) (thickness 0.15)) (justify left bottom) hide)
     )
@@
       (effects (font (size 1.27 1.27) (thickness 0.15)) (justify left bottom) hide)
     )
-    (property "Val" "200R" (at 188.595 53.34 0)
+    (property "Val" "1k" (at 188.595 53.34 0)
       (effects (font (size 1.27 1.27) (thickness 0.15)))
     )
@@
       (effects (font (size 1.27 1.27)) (justify left bottom) hide)
     )
-    (property "LCSC" "C25087" (at 186.055 50.8 0)
+    (property "LCSC" "C11702" (at 186.055 50.8 0)
       (effects (font (size 1.27 1.27)) hide)
     )
@@
       (effects (font (size 1.27 1.27) (thickness 0.15)) hide)
     )
-    (property "Footprint" "LED_SMD:LED_0805_2012Metric" (at 156.845 60.96 0)
+    (property "Footprint" "LED_SMD:LED_0603_1608Metric" (at 156.845 60.96 0)
       (effects (font (size 1.27 1.27) (thickness 0.15)) (justify left bottom) hide)
     )
@@
       (effects (font (size 1.27 1.27) (thickness 0.15)) (justify left bottom) hide)
     )
-    (property "LCSC" "C2296" (at 179.705 50.8 0)
+    (property "LCSC" "C22371297" (at 179.705 50.8 0)
       (effects (font (size 1.27 1.27)) hide)
     )
@@
       (effects (font (size 1.27 1.27)))
     )
-    (property "Value" "200R" (at 111.125 95.25 0)
+    (property "Value" "1k" (at 111.125 95.25 0)
       (effects (font (size 1.27 1.27) (thickness 0.15)) (justify left bottom) hide)
     )
@@
       (effects (font (size 1.27 1.27) (thickness 0.15)) (justify left bottom) hide)
     )
-    (property "Val" "200R" (at 93.345 85.09 0)
+    (property "Val" "1k" (at 93.345 85.09 0)
       (effects (font (size 1.27 1.27) (thickness 0.15)))
     )
@@
       (effects (font (size 1.27 1.27)) (justify left bottom) hide)
     )
-    (property "LCSC" "C25087" (at 90.805 82.55 0)
+    (property "LCSC" "C11702" (at 90.805 82.55 0)
       (effects (font (size 1.27 1.27)) hide)
     )
@@
       (effects (font (size 1.27 1.27) (thickness 0.15)) hide)
     )
-    (property "Footprint" "LED_SMD:LED_0805_2012Metric" (at 160.02 121.285 0)
+    (property "Footprint" "LED_SMD:LED_0603_1608Metric" (at 160.02 121.285 0)
       (effects (font (size 1.27 1.27) (thickness 0.15)) (justify left bottom) hide)
     )
@@
       (effects (font (size 1.27 1.27) (thickness 0.15)) (justify left bottom) hide)
     )
-    (property "LCSC" "C34499" (at 182.88 111.125 0)
+    (property "LCSC" "C5355421" (at 182.88 111.125 0)
       (effects (font (size 1.27 1.27)) hide)
     )
@@
       (effects (font (size 1.27 1.27)))
     )
-    (property "Value" "200R" (at 209.55 123.825 0)
+    (property "Value" "1k" (at 209.55 123.825 0)
       (effects (font (size 1.27 1.27) (thickness 0.15)) (justify left bottom) hide)
     )
@@
       (effects (font (size 1.27 1.27) (thickness 0.15)) (justify left bottom) hide)
     )
-    (property "Val" "200R" (at 191.77 113.665 0)
+    (property "Val" "1k" (at 191.77 113.665 0)
       (effects (font (size 1.27 1.27) (thickness 0.15)))
     )
@@
       (effects (font (size 1.27 1.27)) (justify left bottom) hide)
     )
-    (property "LCSC" "C25087" (at 189.23 111.125 0)
-      (effects (font (size 1.27 1.27)) hide)
-    )
+    (property "LCSC" "C11702" (at 189.23 111.125 0)
+      (effects (font (size 1.27 1.27)) hide)
+    )

Commit message: board drc
Parts:
- D1: value LED_G_0603_LG_L29K-G2J1-24-Z -> LED_B_0603_LG_L29K-G2J1-24-Z
- D2: value LED_G_0603_LG_L29K-G2J1-24-Z -> LED_R_0603_LG_L29K-G2J1-24-Z
- D3: LCSC C22371297 -> C965804
Other:
- note added: "led parts 0603 (2024-09-04): red: C5179624 green: C965804 blue: C5355421"
- note removed: "led parts 0603 (2024-09-04): red: C5179624 green: C22371297 blue: C5355421"
Changed lines of the file:
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@@
     (stroke (width 0) (type default))
   )
-  (text "led parts 0603 (2024-09-04):\nred: C5179624\ngreen: C22371297\nblue: C5355421"
+  (text "led parts 0603 (2024-09-04):\nred: C5179624\ngreen: C965804\nblue: C5355421"
     (at 71.501 62.103 0)
     (effects (font (size 1.27 1.27)) (justify left bottom))
@@
       (effects (font (size 1.27 1.27)))
     )
-    (property "Value" "LED_G_0603_LG_L29K-G2J1-24-Z" (at 61.595 90.17 0)
+    (property "Value" "LED_R_0603_LG_L29K-G2J1-24-Z" (at 61.595 90.17 0)
       (effects (font (size 1.27 1.27) (thickness 0.15)) (justify left bottom) hide)
     )
@@
       (effects (font (size 1.27 1.27) (thickness 0.15)) (justify left bottom) hide)
     )
-    (property "LCSC" "C22371297" (at 179.705 50.8 0)
+    (property "LCSC" "C965804" (at 179.705 50.8 0)
       (effects (font (size 1.27 1.27)) hide)
     )
@@
       (effects (font (size 1.27 1.27)))
     )
-    (property "Value" "LED_G_0603_LG_L29K-G2J1-24-Z" (at 179.07 106.045 0)
+    (property "Value" "LED_B_0603_LG_L29K-G2J1-24-Z" (at 179.07 106.045 0)
       (effects (font (size 1.27 1.27) (thickness 0.15)) hide)
     )

Commit message: board
Parts:
- R33: value 1k -> 510R; LCSC C11702 -> C25123; Val 1k -> 510R
Changed lines of the file:
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@@
       (effects (font (size 1.27 1.27)))
     )
-    (property "Value" "1k" (at 111.125 95.25 0)
+    (property "Value" "510R" (at 111.125 95.25 0)
       (effects (font (size 1.27 1.27) (thickness 0.15)) (justify left bottom) hide)
     )
@@
       (effects (font (size 1.27 1.27) (thickness 0.15)) (justify left bottom) hide)
     )
-    (property "Val" "1k" (at 93.345 85.09 0)
+    (property "Val" "510R" (at 93.345 85.09 0)
       (effects (font (size 1.27 1.27) (thickness 0.15)))
     )
@@
       (effects (font (size 1.27 1.27)) (justify left bottom) hide)
     )
-    (property "LCSC" "C11702" (at 90.805 82.55 0)
+    (property "LCSC" "C25123" (at 90.805 82.55 0)
       (effects (font (size 1.27 1.27)) hide)
     )
