File: boards/nf_ecp5_45/power.kicad_sch (KiCad schematic)
At the start: 39 parts, among them U4 LD1117S18TR_SOT223, U5 TPS62823DLCT, U6 TPS62823DLCT

Commit message: test
Other:
- note added: "TODO: add 0r for vccddr and vccddrref"
Changed lines of the file:
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@@
+    (effects (font (size 1.27 1.27)) (justify left bottom))
+  )
+  (text "TODO: add 0r for vccddr and vccddrref" (at 114.427 40.767 0)
     (effects (font (size 1.27 1.27)) (justify left bottom))
   )

Commit message: board
Parts:
- added R35: 0R, Resistor_SMD:R_0603_1608Metric, symbol Device:R
Connections:
- net VCCDDR3: now also R35.2; no longer C26.2, C32.2, C34.2, L2.2, R20.2, TP4.1
- new net: C26.2, C32.2, C34.2, L2.2, R20.2, R35.1, TP4.1
Changed lines of the file:
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@@
+    (stroke (width 0) (type default))
+  )
+  (wire (pts (xy 149.225 57.785) (xy 152.273 57.785))
     (stroke (width 0) (type default))
   )
@@
     (effects (font (size 1.27 1.27)) (justify left bottom))
   )
-  (global_label "VCCDDR3" (shape output) (at 141.605 57.785 0) (fields_autoplaced)
+  (global_label "VCCDDR3" (shape output) (at 152.273 57.785 0) (fields_autoplaced)
     (effects (font (size 1.27 1.27)) (justify left))
-    (property "Intersheetrefs" "${INTERSHEET_REFS}" (at 153.2383 57.785 0)
+    (property "Intersheetrefs" "${INTERSHEET_REFS}" (at 163.9063 57.785 0)
       (effects (font (size 1.27 1.27)) (justify left) hide)
     )
@@
         )
       )
+    )
+  )
+  (symbol (lib_id "Device:R") (at 145.415 57.785 90) (unit 1)
+    (in_bom yes) (on_board yes) (dnp no) (fields_autoplaced)
+    (property "Reference" "R35" (at 145.415 52.07 90)
+      (effects (font (size 1.27 1.27)))
+    )
+    (property "Value" "0R" (at 145.415 54.61 90)
+      (effects (font (size 1.27 1.27)))
+    )
+    (property "Footprint" "Resistor_SMD:R_0603_1608Metric" (at 145.415 59.563 90)
+      (effects (font (size 1.27 1.27)) hide)
+    )
+    (property "Datasheet" "~" (at 145.415 57.785 0)
+      (effects (font (size 1.27 1.27)) hide)
+    )
+    (property "LCSC" "C100044" (at 145.415 57.785 90)
+      (effects (font (size 1.27 1.27)) hide)
+    )
+    (pin "2")
+    (pin "1")
+    (instances
+      (project "nf_tpu"
+        (path "/9bed7131-c603-46c6-ae3c-0e9faa418ea0/c0b341f4-44f0-405a-beb8-05c2d4a9af1d"
+          (reference "R35") (unit 1)
+        )
+      )

Commit message: board
Parts:
- removed R35: 0R, Resistor_SMD:R_0603_1608Metric, symbol Device:R
Connections:
- net VCCDDR3: now also C26.2, C32.2, C34.2, L2.2, R20.2, TP4.1
Changed lines of the file:
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@@
-    (stroke (width 0) (type default))
-  )
-  (wire (pts (xy 149.225 57.785) (xy 152.273 57.785))
     (stroke (width 0) (type default))
   )
@@
     (stroke (width 0) (type default))
   )
-  (wire (pts (xy 139.065 57.785) (xy 141.605 57.785))
+  (wire (pts (xy 139.065 57.785) (xy 152.273 57.785))
     (stroke (width 0) (type default))
   )
@@
         )
       )
-    )
-  )
-  (symbol (lib_id "Device:R") (at 145.415 57.785 90) (unit 1)
-    (in_bom yes) (on_board yes) (dnp no) (fields_autoplaced)
-    (property "Reference" "R35" (at 145.415 52.07 90)
-      (effects (font (size 1.27 1.27)))
-    )
-    (property "Value" "0R" (at 145.415 54.61 90)
-      (effects (font (size 1.27 1.27)))
-    )
-    (property "Footprint" "Resistor_SMD:R_0603_1608Metric" (at 145.415 59.563 90)
-      (effects (font (size 1.27 1.27)) hide)
-    )
-    (property "Datasheet" "~" (at 145.415 57.785 0)
-      (effects (font (size 1.27 1.27)) hide)
-    )
-    (property "LCSC" "C100044" (at 145.415 57.785 90)
-      (effects (font (size 1.27 1.27)) hide)
-    )
-    (pin "2")
-    (pin "1")
-    (instances
-      (project "nf_tpu"
-        (path "/9bed7131-c603-46c6-ae3c-0e9faa418ea0/c0b341f4-44f0-405a-beb8-05c2d4a9af1d"
-          (reference "R35") (unit 1)
-        )
-      )
