File: boards/nf_art7_100/fpga-ddr.kicad_sch (KiCad schematic)
At the start: 1 part, among them U1 XC7A100T-CSG324

Commit message: art7 io
Other:
- note added: "TODO: connect vref"
Changed lines of the file:
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@@
     (stroke (width 0) (type default))
+  )
+  (text "TODO: connect vref" (at 125.603 46.101 0)
+    (effects (font (size 1.27 1.27)) (justify left bottom))
   )
   (global_label "CK-" (shape input) (at 120.777 126.619 0) (fields_autoplaced)
